File: hardware/smart-knob.kicad_sch (KiCad schematic)
At the start: 0 parts

Commit message: hw: add power power sub-circuit
Parts:
- added C1, C4: 0.1µF, symbol Device:C
- added C2, C5: 10µF, symbol Device:C
- added C3: 4.7nF, symbol Device:C
- added C6, C7: 4.7µF, symbol Device:C
- added D1: LED, symbol Device:LED
- added D2: MBR120VLSFT1G, symbol Device:D_Schottky
- added J1: USB_C_Receptacle_USB2.0_14P, smart-knob:USB_C_Receptacle_HRO_TYPE-C-31-M-12, symbol Connector:USB_C_Receptacle_USB2.0_14P
- added J2: Conn_01x02_Pin, symbol Connector:Conn_01x02_Pin
- added Q1: DMG3415U, symbol Transistor_FET:Q_NMOS_GSD
- added R1, R2: 5.1K, symbol Device:R
- added R3: 1M, symbol Device:R
- added R4: 2K, symbol Device:R
- added R5, R6: 1K, symbol Device:R
- added U1: ESP32-S3-WROOM-1, RF_Module:ESP32-S3-WROOM-1, symbol RF_Module:ESP32-S3-WROOM-1
- added U2: AP2112K-3.3, Package_TO_SOT_SMD:SOT-23-5, symbol Regulator_Linear:AP2112K-3.3
- added U3: MCP73831-2-OT, Package_TO_SOT_SMD:SOT-23-5, symbol Battery_Management:MCP73831-2-OT
Connections:
- new net: D1.2 (A), R5.2
- new net: R4.1, U3.5 (PROG)
- new net: J1.B5 (CC2), R1.1
- new net: J1.A5 (CC1), R2.1
- new net: C3.1, J1.SH (SHIELD), R3.1
- new net: U1.1 (GND), U1.40 (GND), U1.41 (GND)
- new net +3.3V: C4.1, C5.1, U2.5 (VOUT)
- new net +5V: C1.1, C2.1, C6.1, D2.2 (A), J1.A4 (VBUS), J1.A9 (VBUS), J1.B4 (VBUS), J1.B9 (VBUS), Q1.1 (G), R5.1, R6.1, U3.4 (V_{DD})
- new net BAT+: C7.2, J2.1 (Pin_1), Q1.3 (D), U3.3 (V_{BAT})
- new net GND: C1.2, C2.2, C3.2, C4.2, C5.2, C6.2, C7.1, J1.A1 (GND), J1.A12 (GND), J1.B1 (GND), J1.B12 (GND), J2.2 (Pin_2), R1.2, R2.2, R3.2, R4.2, R6.2, U2.2 (GND), U3.2 (V_{SS})
- new net STAT: D1.1 (K), U3.1 (STAT)
- new net USB_D+: J1.A6 (D+), J1.B6 (D+)
- new net USB_D-: J1.A7 (D-), J1.B7 (D-)
- new net VSYS: D2.1 (K), Q1.2 (S), U2.1 (VIN), U2.3 (EN)
Other:
- note added: "USB C & Power"
- company: (none) -> Timothy Kozlowski
- title: (none) -> Smart Knob Hub
